Commit message: 轮子形态+车身大小关联数据修改

File: src/my_nav2_robot/urdf/robot.urdf.xacro (robot description, xacro)
@@ -5,6 +5,6 @@
     <xacro:property name="chassis_width" value="0.3"/>
     <xacro:property name="chassis_height" value="0.1"/>
-    <!--轮子形态-->
-    <xacro:property name="wheel_radius" value="0.05"/>
+    <!--轮子形态（实车机械参数：轮半径 81.5mm）-->
+    <xacro:property name="wheel_radius" value="0.0815"/>
     <xacro:property name="wheel_width" value="0.025"/>
     <!--轮子位置-->

Commit message: little

File: src/my_nav2_robot/urdf/robot.urdf.xacro (robot description, xacro)
@@ -2,5 +2,5 @@
 <robot xmlns:xacro="http://www.ros.org/wiki/xacro" name="my_nav2_bot">
     <!--机器人身体-->
-    <xacro:property name="chassis_length" value="0.4"/>
+    <xacro:property name="chassis_length" value="0.3"/>
     <xacro:property name="chassis_width" value="0.3"/>
     <xacro:property name="chassis_height" value="0.1"/>
@@ -9,6 +9,6 @@
     <xacro:property name="wheel_width" value="0.025"/>
     <!--轮子位置-->
-    <xacro:property name="wheel_offset_x" value="${chassis_length / 2 - 0.05}"/>
-    <xacro:property name="wheel_offset_y" value="${chassis_width / 2 + wheel_width / 2}"/>
+    <xacro:property name="wheel_offset_x" value="${chassis_length / 2}"/>
+    <xacro:property name="wheel_offset_y" value="${chassis_width / 2}"/>
     <xacro:property name="wheel_offset_z" value="-0.02"/>
     <!--机器人机身的物理属性-->

Commit message: little change

File: src/my_nav2_robot/urdf/robot.urdf.xacro (robot description, xacro)
@@ -137,3 +137,17 @@
         <origin xyz="0 0 0" rpy="0 0 0"/>
     </joint>
+    <!--livox lidar-->
+    <link name="livox_frame">
+        <visual>
+            <geometry>
+                <box size="0.06 0.06 0.03"/>
+            </geometry>
+            <material name="red"/>
+        </visual>
+    </link>
+    <joint name="livox_joint" type="fixed">
+        <parent link="base_link"/>
+        <child link="livox_frame"/>
+        <origin xyz="0 0 0.1" rpy="0 0 0"/>
+    </joint>
 </robot>
